File: pcb/radio_solar/radio_solar.sch (KiCad schematic (older format))
At the start: 0 parts

Commit message: Se realiza dibujo inicial del esquematico
Parts:
- added C?: C_Variable, symbol Device:C_Variable
- added C? (x2): C, symbol Device:C
- added C? (x5): CP, symbol Device:CP
- added D?: 1N914, Diode_THT:D_DO-35_SOD27_P7.62mm_Horizontal, symbol Diode:1N914
- added J?: Conn_01x03, symbol Connector_Generic:Conn_01x03
- added J? (x2): Conn_01x02, symbol Connector_Generic:Conn_01x02
- added Q? (x3): BC548, Package_TO_SOT_THT:TO-92_Inline, symbol Transistor_BJT:BC548
- added R? (x6): R, symbol Device:R
- added RV?: R_POT, symbol Device:R_POT
- added SW?: SW_DPST_x2, symbol Switch:SW_DPST_x2
Connections:
- new net: C?.1, J?.3 (Pin_3)
- new net: C?.2, C?.2, C?.2, C?.2, J?.1 (Pin_1), J?.2 (Pin_2), Q?.3 (E), Q?.3 (E), R?.1
- new net: C?.2, D?.1 (K)
- new net: D?.2 (A), J?.2 (Pin_2)
- new net: C?.1, Q?.2 (B), R?.2
- new net: C?.1, R?.1, R?.2, RV?.1
- new net: Q?.1 (C), R?.1, RV?.3
- new net: C?.1, RV?.2
- new net: C?.2, Q?.2 (B), R?.2 (x2)
- new net: C?.1, Q?.1 (C), R?.1, R?.1, R?.1
- new net: C?.1, J?.2 (Pin_2), Q?.1 (C)
- new net: C?.1, Q?.3 (E), R?.2
- new net: C?.1, C?.2, J?.1 (Pin_1), R?.2, SW?.1 (A)
- new net: J?.1 (Pin_1), SW?.2 (B)
